Commit message: bringup package

File: install/scorbot_description/share/scorbot_description/urdf/scorbot_gz_properties.xacro (robot description, xacro)
@@ -2,16 +2,18 @@
 <!--Aqui comienza el robot-->
 <robot name="robot_scorbot" xmlns:xacro="http://ros.org/wiki/xacro" >
-    <!--Cambiar por los eslabones del scorbot-->
     <gazebo reference="base_link">
-        <material>Gazebo/Grey</material>
-    </gazebo>
-    <gazebo reference="link_1">
         <material>Gazebo/Red</material>
     </gazebo>
-    <gazebo reference="link_2">
+    <gazebo reference="Link_1">
+        <material>Gazebo/Orange</material>
+    </gazebo>
+    <gazebo reference="Link_2">
+        <material>Gazebo/Yellow</material>
+    </gazebo>
+    <gazebo reference="Link_3">
+        <material>Gazebo/Green</material>
+    </gazebo>
+    <gazebo reference="Link_4">
         <material>Gazebo/Blue</material>
     </gazebo>
-    <gazebo reference="link_3">
-        <material>Gazebo/Green</material>
-    </gazebo>
 </robot>

Commit message: trajectory controller

File: install/scorbot_description/share/scorbot_description/urdf/scorbot_gz_properties.xacro (robot description, xacro)
@@ -2,4 +2,5 @@
 <!--Aqui comienza el robot-->
 <robot name="robot_scorbot" xmlns:xacro="http://ros.org/wiki/xacro" >
+    <gazebo reference="world"/>
     <gazebo reference="base_link">
         <material>Gazebo/Red</material>

File: install/scorbot_description/share/scorbot_description/urdf/scorbot_urdf.xacro (robot description, xacro)
@@ -1,4 +1,10 @@
 <?xml version="1.0" encoding="utf-8"?>
 <robot name="scorbot" xmlns:xacro="http://ros.org/wiki/xacro" >
+  <link name="world"/>
+  <joint name="joint_world" type="fixed" >
+    <parent link="world" />
+    <child link="base_link" />
+    <origin xyz="0.0 0.0 0.0" rpy="0.0 0.0 0.0" />
+  </joint>
   <link
     name="base_link">

File: install/scorbot_description/share/scorbot_description/urdf/trajectory_controller.xacro (robot description, xacro)
@@ -6,9 +6,9 @@
             <plugin>gazebo_ros2_control/GazeboSystem</plugin>
         </hardware>
+        <joint name="joint_world"/>
         <joint name="joint_1">
             <command_interface name="position"/>
             <state_interface name="position"/>
             <state_interface name="velocity"/>
-            <!--<state_interface name="effort"/>-->
         </joint>
         <joint name="joint_2">
@@ -16,5 +16,4 @@
             <state_interface name="position"/>
             <state_interface name="velocity"/>
-            <!--<state_interface name="effort"/>-->
         </joint>
         <joint name="joint_3">
@@ -22,5 +21,4 @@
             <state_interface name="position"/>
             <state_interface name="velocity"/>
-            <!--<state_interface name="effort"/>-->
         </joint>
         <joint name="joint_4">
@@ -28,5 +26,4 @@
             <state_interface name="position"/>
             <state_interface name="velocity"/>
-            <!--<state_interface name="effort"/>-->
         </joint>
     </ros2_control>
